File: JaysCarECUAdapter/JaysCarECUAdapter.brd (EAGLE design)
At the start: 167.3 x 87.6 mm, 2 parts

Commit message: Switched to a smaller board, completed the routing.
Parts:
- moved U$1 103.6 mm to (31.8, 26.7), turned to 180 degrees
- moved U$2 102.2 mm to (31.8, 6.35)
Connections:
- new net N$10: U$1.17, U$2.14
- new net N$11: U$1.16, U$2.13
- new net N$12: U$1.18, U$2.15
- new net N$13: U$1.14, U$2.17
- new net N$14: U$1.13, U$2.16
- new net N$15: U$1.15, U$2.18
- new net N$16: U$1.11, U$2.20
- new net N$17: U$1.10, U$2.19
- new net N$18: U$1.12, U$2.21
- new net N$19: U$1.8, U$2.23
- new net N$20: U$1.9, U$2.24
- new net N$21: U$1.7, U$2.22
- new net N$22: U$1.5, U$2.26
- new net N$23: U$1.4, U$2.25
- new net N$24: U$1.6, U$2.27
- new net N$25: U$1.2, U$2.29
- new net N$26: U$1.3, U$2.30
- new net N$27: U$1.1, U$2.28
- new net N$28: U$1.28, U$2.1
- new net N$29: U$1.29, U$2.2
- new net N$30: U$1.30, U$2.3
- new net N$5: U$1.24, U$2.9
- new net N$6: U$1.22, U$2.7
- new net N$7: U$1.20, U$2.11
- new net N$8: U$1.19, U$2.10
- new net N$9: U$1.21, U$2.12
- net N$1: now also U$1.26, U$2.5; no longer U$1.1, U$2.60
- net N$2: now also U$1.27, U$2.6; no longer U$1.30, U$2.31
- net N$3: now also U$1.25, U$2.4; no longer U$1.31, U$2.30
- net N$4: now also U$1.23, U$2.8; no longer U$1.60, U$2.1
Routing:
- net N$30: track 0.00 -> 33.9 mm
- net N$15: track 0.00 -> 33.8 mm
- net N$26: track 0.00 -> 33.7 mm
- net N$12: track 0.00 -> 33.2 mm
- net N$9: track 0.00 -> 30.3 mm
- net N$18: track 0.00 -> 30.1 mm
- net N$24: track 0.00 -> 29.8 mm
- net N$20: track 0.00 -> 29.7 mm
- net N$2: track 0.00 -> 29.7 mm
- net N$5: track 0.00 -> 29.6 mm
- net N$25: track 0.00 -> 23.5 mm
- net N$29: track 0.00 -> 23.0 mm
- net N$10: track 0.00 -> 22.9 mm
- net N$13: track 0.00 -> 22.9 mm
- net N$22: track 0.00 -> 22.3 mm
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Other:
- board size 167.3 x 87.6 mm -> 64.4 x 33 mm
- board text added: "Nick Butts Car ECU Adapter V1.0"
