File: POVDisplayBase/POVDisplayBase.brd (EAGLE design)
At the start: 80 x 99 mm, 20 parts, among them IC2 NE555D, J1 DCJ0202, Q2 FQD10N20L

Commit message: Updated the POVBase to use a PSoC, it is about the same price as a 555 and more flexible.
Parts:
- removed C6: 15p, resistor:C0603
- removed IC2: NE555D, linear:SO08
- removed R11: 3, resistor:R1210
- removed R5: 100, pot:3223J
- removed R9: 10K, resistor:R0603
- added C3: 10u, resistor:C0603
- added IC1: LD117AS12TR, v-reg:SOT223
- added LED2: LTST-C19HE1WT, NicksParts:LTST-C19HE1WT
- added R1: 0, resistor:R0603
- added R2: 200, resistor:R0603
- added R6: 360, resistor:R0603
- added SV1: (no value), con-lstb:MA05-1
- added U1: CY8C4013SXI-400, NicksParts:SOIC08
- C2: value DNP -> 0.1u
- R3: value 0 -> 10K
- R7: value 100 -> 120; device pot:3223J -> resistor:R0603
- R8: value 200 -> 10K
- moved R3 42.6 mm to (34.1, 9.89)
- moved SL1 36.2 mm to (5.73, 3.00)
- moved SL2 36.2 mm to (41.9, 3.81)
- moved R7 14.2 mm to (63.5, 2.54), turned to 0 degrees
- moved S1 14.0 mm to (30.5, 3.81)
- moved S2 14.0 mm to (16.5, 3.81)
- moved C2 5.61 mm to (55.4, 10.5)
- moved R8 2.54 mm to (47.0, 17.8), turned to 90 degrees
- renumbered C10 to C1, D3 to D2, Q2 to Q1, R10 to R4
Connections:
- removed net N$12: D2.C, R11.2
- removed net N$14: C2.1, IC2.5
- removed net N$9: IC2.7, R5.3, R7.3
- removed net NE555_OUT: IC2.3, S2.3
- new net COIL_DR: S1.3, U1.7
- new net LED: R8.1, U1.2
- new net N$6: LED2.A, R8.2
- new net N$7: C2.1, U1.3
- new net SWDCLK: SV1.4, U1.1
- new net SWDIO: SV1.5, U1.8
- new net TX: SV1.3, U1.6
- new net VCC: C3.1, IC1.4, R7.1, SV1.1, U1.4
- net +12V: now also IC1.3, R2.2, S2.2; no longer IC2.4, IC2.8, R7.2, R8.2, S1.2
- net CONNECTED: now also R1.1; no longer R3.1
- net GND: now also LED2.RED, R1.2, R6.2, SV1.2, U1.5; no longer C6.2, IC2.1, R9.2
- net N$13: now also S1.1, SL2.2; no longer S2.1, SL1.2
- net N$2: now also R2.1; no longer R8.1
- net N$3: now also S2.3, SL1.2; no longer S1.3, SL2.2
- net N$5: now also C3.2, IC1.1, R6.1, R7.2; no longer C6.1, IC2.2, IC2.6, R5.2
- net POS_COIL: now also D2.C; no longer R11.1
- net PWR_TRANSFER: now also R3.1, S1.2; no longer R9.1, S2.2
Routing:
- net N$8: track 2975.2 -> 0.00 mm, vias 2 -> 0
- net NEG_COIL: track 50.6 -> 3025.9 mm, vias 2 -> 4
- net N$9: track 32.3 -> 0.00 mm, vias 2 -> 0
- net NE555_OUT: track 25.7 -> 0.00 mm
- net POS_COIL: track 45.2 -> 70.4 mm
- net VCC: track 0.00 -> 23.8 mm
- net COIL_DR: track 0.00 -> 23.0 mm
- net TX: track 0.00 -> 15.3 mm, vias 0 -> 1
- net N$5: track 17.0 -> 6.69 mm
- net LED: track 0.00 -> 9.87 mm
- net SWDCLK: track 0.00 -> 7.73 mm
- net SWDIO: track 0.00 -> 7.73 mm
- net +12V: track 75.4 -> 69.1 mm
- net N$14: track 5.09 -> 0.00 mm
- net N$12: track 3.90 -> 0.00 mm
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- added copper zone on layer 1, net NEG_COIL

Commit message: Order Oshpark boards for POV Rotate and POV Base
Other:
- board text added: "POVDisplayBaseV3 Nick Butts 2016"
- board text removed: "POVDisplayBaseV2 Nick Butts 2016"
Changed lines of the file:
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@@
 <hole x="75.3" y="24.7" drill="5"/>
 <circle x="72" y="1" radius="0.316225" width="0.254" layer="16"/>
-<text x="27.94" y="93.98" size="1.778" layer="25" font="vector" ratio="15">POVDisplayBaseV2
+<text x="27.94" y="93.98" size="1.778" layer="25" font="vector" ratio="15">POVDisplayBaseV3
 Nick Butts 2016</text>
 <text x="6" y="6" size="0.8128" layer="25" font="vector" ratio="15">FAN+</text>
