File: POVDisplayRotate/POVDisplayRotate.brd (EAGLE design)
At the start: 52 x 86 mm, 49 parts, among them U1 STP08DP05, U2 STP08DP05, U3 MPQ4420Q, U4 CY8CKIT-142, U5 M95M01

Commit message: Updated Abercrombie values.
Routing:
- net GND: track 22.6 -> 41.0 mm, vias 1 -> 5
- net RLED2: track 20.0 -> 25.6 mm
- net BLED1: track 25.2 -> 30.8 mm, vias 2 -> 0
- net GLED1: track 20.8 -> 25.1 mm, vias 2 -> 0
- net SCLK: track 101.6 -> 105.7 mm, vias 2 -> 6
- net RLED1: track 21.0 -> 22.5 mm, vias 2 -> 0
- net SDI: track 70.6 -> 69.3 mm
